Commit message: Primer commit - paquete lesson_urdf funcional en RViz

File: urdf/planar_3dof.urdf (robot description, URDF)
Before this commit: robot planar_3dof, 6 links, 5 joints
Links:
- removed link end
- added link link_twist_mount
- link base_link: geometry visual mesh filename=package://lesson_urdf/meshes/visual/arm_link.stl scale=1 1 1
- link gripper: mass 1 -> None; geometry 
- link link_1: mass 1 -> None; geometry visual mesh filename=package://lesson_urdf/meshes/visual/arm_link.stl scale=1 1 1
- link link_2: mass 1 -> None; geometry visual mesh filename=package://lesson_urdf/meshes/visual/arm_link.stl scale=1 1 1
Joints:
- removed joint gripper_end
- added joint joint_gripper_fixed: type fixed, parent link_2, child gripper, origin xyz=0.5 0.0 0.0 rpy=0 0 0
- joint joint_1: axis 0 0 1 -> 0 1 0; child link_1 -> link_twist_mount; origin xyz=0 0 0.05 rpy=0 0 0 -> xyz=0.0 0.0 0.12 rpy=0 0 0
- joint joint_2: child link_2 -> link_1; origin xyz=0.5 0.0 0.0 rpy=0.0 0 0.0 -> xyz=0.0 0.0 0.0 rpy=0 0 0; parent link_1 -> link_twist_mount
- joint joint_3: child gripper -> link_2; origin xyz=0.5 0.0 0.0 rpy=0.0 0 0.0 -> xyz=0.5 0.0 0.0 rpy=0 0 0; parent link_2 -> link_1
