Commit message: Gazebo and Rviz

File: urdf/legrobot.urdf (robot description, URDF)
Before this commit: robot legrobot, 5 links, 4 joints
Links:
- removed link foot_link
- removed link link_c
- removed link link_p
- removed link link_r
- added link Link_c_left, mass 119.7; collision mesh filename=package://lesson_urdf/meshes/Link_c_left.STL; visual mesh filename=package://lesson_urdf/meshes/Link_c_left.STL
- added link Link_c_right, mass 119.7; collision mesh filename=package://lesson_urdf/meshes/Link_c_right.STL; visual mesh filename=package://lesson_urdf/meshes/Link_c_right.STL
- added link Link_p_left, mass 505.3; collision mesh filename=package://lesson_urdf/meshes/Link_p_left.STL; visual mesh filename=package://lesson_urdf/meshes/Link_p_left.STL
- added link Link_p_right, mass 505.3; collision mesh filename=package://lesson_urdf/meshes/Link_p_right.STL; visual mesh filename=package://lesson_urdf/meshes/Link_p_right.STL
- added link Link_r_left, mass 497.35; collision mesh filename=package://lesson_urdf/meshes/Link_r_left.STL; visual mesh filename=package://lesson_urdf/meshes/Link_r_left.STL
- added link Link_r_right, mass 497.35; collision mesh filename=package://lesson_urdf/meshes/Link_r_right.STL; visual mesh filename=package://lesson_urdf/meshes/Link_r_right.STL
- link base_link: mass 27.938 -> 505.3
Joints:
- removed joint joint_c
- removed joint joint_foot
- removed joint joint_p
- removed joint joint_r
- added joint Joint_c_left: type revolute, parent base_link, child Link_c_left, origin xyz=0 0.8 0 rpy=1.5708 0 1.5708, axis 0 0 1, limit lower=-1.5708 upper=1.5708 effort=100 velocity=5
- added joint Joint_c_right: type revolute, parent base_link, child Link_c_right, origin xyz=0 -0.8 0 rpy=1.5708 0 1.5708, axis 0 0 1, limit lower=-1.5708 upper=1.5708 effort=100 velocity=5
- added joint Joint_p_left: type revolute, parent Link_c_left, child Link_p_left, origin xyz=-0.00013659 -0.099312 0.25 rpy=1.5708 0 -0.0013754, axis 0 0 1, limit lower=-1.5708 upper=1.5708 effort=100 velocity=5
- added joint Joint_p_right: type revolute, parent Link_c_right, child Link_p_right, origin xyz=-0.00013659 -0.099312 0.25 rpy=1.5708 0 -0.0013754, axis 0 0 1, limit lower=-1.5708 upper=1.5708 effort=100 velocity=5
- added joint Joint_r_left: type revolute, parent Link_p_left, child Link_r_left, origin xyz=0 1.6 0 rpy=-3.1416 0 0, axis 0 0 1, limit lower=-1.5708 upper=1.5708 effort=100 velocity=5
- added joint Joint_r_right: type revolute, parent Link_p_right, child Link_r_right, origin xyz=0 1.6 0 rpy=3.1416 0 0, axis 0 0 1, limit lower=-1.5708 upper=1.5708 effort=100 velocity=5

File: urdf/planar_3dof.urdf.xacro (robot description, xacro)
@@ -18,5 +18,5 @@
     <inertial>
       <origin xyz="-0.24659 0 0" rpy="0 0 0"/>
-      <mass value="505.3"/>
+      <mass value="11.35"/>
       <inertia ixx="180.49" ixy="0" ixz="0"
                iyy="21.405" iyz="0" izz="181.05"/>
@@ -50,5 +50,5 @@
       </collision>
       <inertial>
-        <mass value="1.0"/>
+        <mass value="5.0"/>
         <origin xyz="0 0 0"/>
         <inertia ixx="0.01" iyy="0.01" izz="0.01"
@@ -61,5 +61,5 @@
       <child link="Link_c_${side}"/>
       <axis xyz="0 0 1"/>
-      <limit lower="-1.57" upper="1.57" effort="100" velocity="5"/>
+      <limit lower="-1.5708" upper="1.5708" effort="100" velocity="5"/>  <!-- Restricted to ±90° -->
     </joint>
     <gazebo reference="Joint_c_${side}">
@@ -79,5 +79,5 @@
       </collision>
       <inertial>
-        <mass value="1.0"/>
+        <mass value="15.0"/>
         <origin xyz="0 0 0"/>
         <inertia ixx="0.01" iyy="0.01" izz="0.01"
@@ -90,5 +90,5 @@
       <child link="Link_p_${side}"/>
       <axis xyz="0 0 1"/>
-      <limit lower="-1.57" upper="1.57" effort="100" velocity="5"/>
+      <limit lower="-1.5708" upper="1.5708" effort="100" velocity="5"/>  <!-- Restricted to ±90° -->
     </joint>
     <gazebo reference="Joint_p_${side}">
@@ -108,5 +108,5 @@
       </collision>
       <inertial>
-        <mass value="1.0"/>
+        <mass value="8.0"/>
         <origin xyz="0 0 0"/>
         <inertia ixx="0.01" iyy="0.01" izz="0.01"
@@ -119,5 +119,5 @@
       <child link="Link_r_${side}"/>
       <axis xyz="0 0 1"/>
-      <limit lower="-1.57" upper="1.57" effort="100" velocity="5"/>
+      <limit lower="-1.5708" upper="1.5708" effort="100" velocity="5"/>  <!-- Restricted to ±90° -->
     </joint>
     <gazebo reference="Joint_r_${side}">
