Commit message: Simulación Prototipo Control

File: urdf/planar_3dof.urdf.xacro (robot description, xacro)
@@ -1,142 +1,375 @@
 <?xml version="1.0"?>
-<robot name="planar_3dof" xmlns:xacro="http://www.ros.org/wiki/xacro">
-  <!-- ========================= -->
-  <!-- ARGUMENTS -->
-  <!-- ========================= -->
+<robot name="planar_3dof_full" xmlns:xacro="http://www.ros.org/wiki/xacro">
+  <!-- =====================================================
+                            ARGUMENTS
+       ===================================================== -->
   <xacro:arg name="pkg_share" default=""/>
   <xacro:arg name="controllers_yaml" default=""/>
-  <xacro:arg name="mesh_scale" default="1 1 1"/>
-  <xacro:arg name="fix_to_world" default="false"/>
   <xacro:property name="pkg_share" value="$(arg pkg_share)"/>
   <xacro:property name="controllers_yaml" value="$(arg controllers_yaml)"/>
-  <xacro:property name="mesh_scale" value="$(arg mesh_scale)"/>
-  <xacro:property name="fix_to_world" value="$(arg fix_to_world)"/>
-  <!-- ========================= -->
-  <!-- BASE LINK -->
-  <!-- ========================= -->
+  <!-- =====================================================
+                       WORLD (Debugging)
+       ===================================================== -->
+<!--  <link name="world"/>
+  <joint name="world_to_base" type="fixed">
+    <parent link="world"/>
+    <child link="base_link"/>
+    <origin xyz="0 0 0.5" rpy="1.5708 0 0"/>
+  </joint> -->
+  <!-- =====================================================
+                            BASE LINK
+       ===================================================== -->
   <link name="base_link">
     <inertial>
-      <origin xyz="-0.24659 0 0" rpy="0 0 0"/>
-      <mass value="11.35"/>
-      <inertia ixx="180.49" ixy="0" ixz="0"
-               iyy="21.405" iyz="0" izz="181.05"/>
-    </inertial>
-    <visual>
-      <geometry>
-        <mesh filename="file://${pkg_share}/meshes/base_link.STL"/>
-      </geometry>
-    </visual>
-    <collision>
-      <geometry>
-        <mesh filename="file://${pkg_share}/meshes/base_link.STL"/>
-      </geometry>
-    </collision>
-  </link>
-  <!-- ========================= -->
-  <!-- LEG MACRO -->
-  <!-- ========================= -->
-  <xacro:macro name="leg" params="side parent y_offset rpy_c rpy_r">
-    <!-- C LINK -->
-    <link name="Link_c_${side}">
-      <visual>
-        <geometry>
-          <mesh filename="file://${pkg_share}/meshes/Link_c_${side}.STL"/>
-        </geometry>
-      </visual>
-      <collision>
-        <geometry>
-          <mesh filename="file://${pkg_share}/meshes/Link_c_${side}.STL"/>
-        </geometry>
-      </collision>
-      <inertial>
-        <mass value="5.0"/>
-        <origin xyz="0 0 0"/>
-        <inertia ixx="0.01" iyy="0.01" izz="0.01"
-                 ixy="0" ixz="0" iyz="0"/>
-      </inertial>
-    </link>
-    <joint name="Joint_c_${side}" type="revolute">
-      <origin xyz="0 ${y_offset} 0" rpy="${rpy_c}"/>
-      <parent link="${parent}"/>
-      <child link="Link_c_${side}"/>
-      <axis xyz="0 0 1"/>
-      <limit lower="-1.5708" upper="1.5708" effort="100" velocity="5"/>  <!-- Restricted to ±90° -->
-    </joint>
-    <gazebo reference="Joint_c_${side}">
-      <provideFeedback>true</provideFeedback>
-    </gazebo>
-    <!-- P LINK -->
-    <link name="Link_p_${side}">
-      <visual>
-        <geometry>
-          <mesh filename="file://${pkg_share}/meshes/Link_p_${side}.STL"/>
-        </geometry>
-      </visual>
-      <collision>
-        <geometry>
-          <mesh filename="file://${pkg_share}/meshes/Link_p_${side}.STL"/>
-        </geometry>
-      </collision>
-      <inertial>
-        <mass value="15.0"/>
-        <origin xyz="0 0 0"/>
-        <inertia ixx="0.01" iyy="0.01" izz="0.01"
-                 ixy="0" ixz="0" iyz="0"/>
-      </inertial>
-    </link>
-    <joint name="Joint_p_${side}" type="revolute">
-      <origin xyz="-0.00013659 -0.099312 0.25" rpy="1.5708 0 -0.0013754"/>
-      <parent link="Link_c_${side}"/>
-      <child link="Link_p_${side}"/>
-      <axis xyz="0 0 1"/>
-      <limit lower="-1.5708" upper="1.5708" effort="100" velocity="5"/>  <!-- Restricted to ±90° -->
-    </joint>
-    <gazebo reference="Joint_p_${side}">
-      <provideFeedback>true</provideFeedback>
-    </gazebo>
-    <!-- R LINK -->
-    <link name="Link_r_${side}">
-      <visual>
-        <geometry>
-          <mesh filename="file://${pkg_share}/meshes/Link_r_${side}.STL"/>
-        </geometry>
-      </visual>
-      <collision>
-        <geometry>
-          <mesh filename="file://${pkg_share}/meshes/Link_r_${side}.STL"/>
-        </geometry>
-      </collision>
-      <inertial>
-        <mass value="8.0"/>
-        <origin xyz="0 0 0"/>
-        <inertia ixx="0.01" iyy="0.01" izz="0.01"
-                 ixy="0" ixz="0" iyz="0"/>
-      </inertial>
-    </link>
-    <joint name="Joint_r_${side}" type="revolute">
-      <origin xyz="0 1.6 0" rpy="${rpy_r}"/>
-      <parent link="Link_p_${side}"/>
-      <child link="Link_r_${side}"/>
-      <axis xyz="0 0 1"/>
-      <limit lower="-1.5708" upper="1.5708" effort="100" velocity="5"/>  <!-- Restricted to ±90° -->
-    </joint>
-    <gazebo reference="Joint_r_${side}">
-      <provideFeedback>true</provideFeedback>
-    </gazebo>
-  </xacro:macro>
-  <!-- ========================= -->
-  <!-- LEGS -->
-  <!-- ========================= -->
-  <xacro:leg side="right" parent="base_link"
-             y_offset="-0.8"
-             rpy_c="1.5708 0 1.5708"
-             rpy_r="3.1416 0 0"/>
-  <xacro:leg side="left" parent="base_link"
-             y_offset="0.8"
-             rpy_c="1.5708 0 1.5708"
-             rpy_r="-3.1416 0 0"/>
-  <!-- ========================= -->
-  <!-- ROS2 CONTROL -->
-  <!-- ========================= -->
+      <origin xyz="0 0 0" rpy="0 0 0"/>
+      <mass value="0.240693"/>
+      <inertia
+        ixx="0.001"
+        iyy="0.001"
+        izz="0.001"
+        ixy="0"
+        ixz="0"
+        iyz="0"/>
+    </inertial>
+    <visual>
+      <geometry>
+        <mesh filename="file://${pkg_share}/meshes/base_link.STL"
+              scale="1 1 1"/>
+      </geometry>
+    </visual>
+    <collision>
+      <geometry>
+        <mesh filename="file://${pkg_share}/meshes/base_link.STL"
+              scale="1 1 1"/>
+      </geometry>
+    </collision>
+  </link>
+  <!-- =====================================================
+                            LEFT LEG
+       ===================================================== -->
+  <link name="Link_c_left">
+    <inertial>
+      <origin xyz="0 0 0" rpy="0 0 0"/>
+      <mass value="0.076578"/>
+      <inertia
+        ixx="0.0005"
+        iyy="0.0005"
+        izz="0.0005"
+        ixy="0"
+        ixz="0"
+        iyz="0"/>
+    </inertial>
+    <visual>
+      <geometry>
+        <mesh filename="file://${pkg_share}/meshes/Link_c_left.STL"
+              scale="1 1 1"/>
+      </geometry>
+    </visual>
+    <collision>
+      <geometry>
+        <mesh filename="file://${pkg_share}/meshes/Link_c_left.STL"
+              scale="1 1 1"/>
+      </geometry>
+    </collision>
+  </link>
+  <joint name="Joint_c_left" type="revolute">
+    <origin xyz="0.0803 0 0" rpy="0 0 0"/>
+    <parent link="base_link"/>
+    <child link="Link_c_left"/>
+    <axis xyz="0 0 1"/>
+    <limit
+      lower="-1.5708"
+      upper="1.5708"
+      effort="1000"
+      velocity="2"/>
+    <dynamics
+      damping="300.0"
+      friction="100.0"/>
+  </joint>
+  <link name="Link_p_left">
+    <inertial>
+      <origin xyz="0 0 0" rpy="0 0 0"/>
+      <mass value="0.27292"/>
+      <inertia
+        ixx="0.001"
+        iyy="0.001"
+        izz="0.001"
+        ixy="0"
+        ixz="0"
+        iyz="0"/>
+    </inertial>
+    <visual>
+      <geometry>
+        <mesh filename="file://${pkg_share}/meshes/Link_p_left.STL"
+              scale="1 1 1"/>
+      </geometry>
+    </visual>
+    <collision>
+      <geometry>
+        <mesh filename="file://${pkg_share}/meshes/Link_p_left.STL"
+              scale="1 1 1"/>
+      </geometry>
+    </collision>
+  </link>
+  <joint name="Joint_p_left" type="revolute">
+    <origin xyz="0.0705 -0.017147 -0.00786"
+            rpy="0 -1.5708 0"/>
+    <parent link="Link_c_left"/>
+    <child link="Link_p_left"/>
+    <axis xyz="0 0 -1"/>
+    <limit
+      lower="-1.5708"
+      upper="1.5708"
+      effort="1000"
+      velocity="2"/>
+    <dynamics
+      damping="300.0"
+      friction="100.0"/>
+  </joint>
+  <link name="Link_r_left">
+    <inertial>
+      <origin xyz="0 0 0" rpy="0 0 0"/>
+      <mass value="0.096277"/>
+      <inertia
+        ixx="0.0005"
+        iyy="0.0005"
+        izz="0.0005"
+        ixy="0"
+        ixz="0"
+        iyz="0"/>
+    </inertial>
+    <visual>
+      <geometry>
+        <mesh filename="file://${pkg_share}/meshes/Link_r_left.STL"
+              scale="1 1 1"/>
+      </geometry>
+    </visual>
+    <collision>
+      <geometry>
+        <mesh filename="file://${pkg_share}/meshes/Link_r_left.STL"
+              scale="1 1 1"/>
+      </geometry>
+    </collision>
+  </link>
+  <joint name="Joint_r_left" type="revolute">
+    <origin xyz="0 -0.13069 0"
+            rpy="3.129 -0.00050149 -0.03981"/>
+    <parent link="Link_p_left"/>
+    <child link="Link_r_left"/>
+    <axis xyz="0 0 1"/>
+    <limit
+      lower="-1.5708"
+      upper="1.5708"
+      effort="1000"
+      velocity="2"/>
+    <dynamics
+      damping="300.0"
+      friction="100.0"/>
+  </joint>
+  <link name="Link_wheels_left">
+    <inertial>
+      <origin xyz="0 0 -0.013" rpy="0 0 0"/>
+      <mass value="0.065044"/>
+      <inertia
+        ixx="2.77E-05"
+        iyy="2.77E-05"
+        izz="4.9085E-05"
+        ixy="0"
+        ixz="0"
+        iyz="0"/>
+    </inertial>
+    <visual>
+      <geometry>
+        <mesh filename="file://${pkg_share}/meshes/Link_wheels_left.STL"
+              scale="1 1 1"/>
+      </geometry>
+    </visual>
+    <collision>
+      <geometry>
+        <mesh filename="file://${pkg_share}/meshes/Link_wheels_left.STL"
+              scale="1 1 1"/>
+      </geometry>
+    </collision>
+  </link>
+  <joint name="Joint_wheels_left" type="continuous">
+    <origin
+      xyz="0.0049779 0.13502 0.0082029"
+      rpy="0.0126 0 -0.039813"/>
+    <parent link="Link_r_left"/>
+    <child link="Link_wheels_left"/>
+    <axis xyz="0 0 1"/>
+    <limit
+      effort="1000"
+      velocity="20"/>
+    <dynamics
+      damping="3.0"
+      friction="0.1"/>
+  </joint>
+  <!-- =====================================================
+                           RIGHT LEG
+       ===================================================== -->
+  <link name="Link_c_right">
+    <inertial>
+      <origin xyz="0 0 0" rpy="0 0 0"/>
+      <mass value="0.077224"/>
+      <inertia
+        ixx="0.0005"
+        iyy="0.0005"
+        izz="0.0005"
+        ixy="0"
+        ixz="0"
+        iyz="0"/>
+    </inertial>
+    <visual>
+      <geometry>
+        <mesh filename="file://${pkg_share}/meshes/Link_c_right.STL"
+              scale="1 1 1"/>
+      </geometry>
+    </visual>
+    <collision>
+      <geometry>
+        <mesh filename="file://${pkg_share}/meshes/Link_c_right.STL"
+              scale="1 1 1"/>
+      </geometry>
+    </collision>
+  </link>
+  <joint name="Joint_c_right" type="revolute">
+    <origin xyz="0 0 0" rpy="0 0 0"/>
+    <parent link="base_link"/>
+    <child link="Link_c_right"/>
+    <axis xyz="0 0 1"/>
+    <limit
+      lower="-1.5708"
+      upper="1.5708"
+      effort="1000"
+      velocity="5"/>
+    <dynamics
+      damping="100.0"
+      friction="50.0"/>
+  </joint>
+  <link name="Link_p_right">
+    <inertial>
+      <origin xyz="0 0 0" rpy="0 0 0"/>
+      <mass value="0.27292"/>
+      <inertia
+        ixx="0.001"
+        iyy="0.001"
+        izz="0.001"
+        ixy="0"
+        ixz="0"
+        iyz="0"/>
+    </inertial>
+    <visual>
+      <geometry>
+        <mesh filename="file://${pkg_share}/meshes/Link_p_right.STL"
+              scale="1 1 1"/>
+      </geometry>
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