Commit message: Actualización URDF y ajustes en joint_gui

File: lesson_urdf-main/urdf/Pierna enteraaaaaaaaaaa.SLDASM.urdf (robot description, URDF)
Before this commit: robot Pierna_entera_2, 4 links, 3 joints
Links:
- link base_link: mass 0.313191197329196 -> 0.31319
- link link_c: mass 0.30893 -> 0.3089298949799
- link link_p: mass 0.13838 -> 0.138380104137137
- link link_r: mass 0.1843 -> 0.184300341408798
Joints:
- joint joint_c: origin xyz=-0.0047758 0.041904 0.02325 rpy=1.5708 0 -3.0281 -> xyz=0.0021041 0.042122 0.02325 rpy=1.5708 0 3.0917
- joint joint_r: origin xyz=0.44154 0.15513 0.037775 rpy=0 0 0 -> xyz=0.468 0 0.037775 rpy=0 0 0
