Commit message: Gazebo y joint_gui modificado

File: lesson_urdf-main/urdf/legrobot.urdf (robot description, URDF)
Before this commit: robot Pierna enteraaaaaaaaaaa.SLDASM, 4 links, 3 joints
Links:
- added link foot_link; visual sphere radius=0.01
Joints:
- added joint joint_foot: type fixed, parent link_r, child foot_link, origin xyz=0.441000 0.0 -0.0117 rpy=0 0 0

Commit message: Nuevo URDF actualizado y método geométrico de cinemática directa

File: lesson_urdf-main/urdf/legrobot.urdf (robot description, URDF)
Before this commit: robot legrobot, 5 links, 4 joints
Links:
- link base_link: mass 0.31319 -> 27.938
- link link_c: mass 0.3089298949799 -> 0.395989033420963
- link link_p: mass 0.138380104137137 -> 0.44537879484085
- link link_r: mass 0.184300341408798 -> 0.154972710016794
Joints:
- joint joint_c: axis 0 0 -1 -> 0 0 1; limit (none) -> lower=-1.571 upper=1.571 effort=0 velocity=0; origin xyz=0.0021041 0.042122 0.02325 rpy=1.5708 0 3.0917 -> xyz=0 0 0 rpy=0 0 0; parent link_p -> base_link; type continuous -> revolute
- joint joint_foot: origin xyz=0.441000 0.0 -0.0117 rpy=0 0 0 -> xyz=0.16093478 0.00001944 0.03845750 rpy=0 0 0
- joint joint_p: axis 0 0 1 -> 0 0 -1; limit (none) -> lower=-1.571 upper=1.571 effort=0 velocity=0; origin xyz=-0.0024512 -0.097818 0.25643 rpy=1.5091 0 -3.1416 -> xyz=-0.018425 -7.5056E-05 0.0728 rpy=1.5708 0 -1.5708; parent base_link -> link_c; type continuous -> revolute
- joint joint_r: limit (none) -> lower=-1.571 upper=1.571 effort=0 velocity=0; origin xyz=0.468 0 0.037775 rpy=0 0 0 -> xyz=0.18787 0 0.064085 rpy=0 0 0; parent link_c -> link_p; type continuous -> revolute
